File: ECE4760 Motor Driver.kicad_pcb (KiCad board)
At the start: 6 copper layers, 43.2 x 45.7 mm, 144 parts, among them J1 IO, J100 Alternative Motor, J2 Motor / Power, J3 USB_B_Micro, J4 UART, J5 Debug, J6 Boot, Q1 EPC23104, Q2 EPC23104, Q3 EPC23104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

Commit message: Getting ready for fab
Parts:
- added TP5: TestPoint, TestPoint:TestPoint_Pad_D2.0mm, B.Cu at (106.9, 55.4)
- C38, C39, C40, C41, C42, C43, C44, C45, C46, C47, C48, C49, C50, C51, C52, C53: value 1u, 100V -> 100n, 100V, 0603, X7R
- C54, C55, C56, C57, C58, C59, C60, C61, C62, C63, C64, C65: value 1u, 100V -> 1u, 100V, 0805, X7R
- R2, R3: value 5k -> 1k
Routing:
- net GND: vias 199 -> 200
Other:
- board text added: "ECE4760 Motor Driver SJB / 2023 rev 0"

Commit message: Play around with switching to RP2040
Parts:
- removed U1: STM32G473V_B-C-E_Hx, Package_BGA:TFBGA-100_8x8mm_Layout10x10_P0.8mm
- removed X1: 48MHz, Oscillator:Oscillator_SMD_ECS_2520MV-xxx-xx-4Pin_2.5x2.0mm
- added C74: 100n, Capacitor_SMD:C_0402_1005Metric, F.Cu at (65.4, 57.1)
- added C75: 100n, Capacitor_SMD:C_0402_1005Metric, F.Cu at (64.1, 54.7)
- added C76: 100n, Capacitor_SMD:C_0402_1005Metric, F.Cu at (63.1, 54.7)
- added C77: 100n, Capacitor_SMD:C_0402_1005Metric, F.Cu at (62.1, 54.7)
- added C78: 100n, Capacitor_SMD:C_0402_1005Metric, F.Cu at (60.5, 54.7)
- added C79: 100n, Capacitor_SMD:C_0402_1005Metric, F.Cu at (59.5, 54.7)
- added U10: W25Q32JVSS, W25Q:W25Q64JWUUIQTR, F.Cu at (56.5, 52.7)
- added U7: RP2040, Package_DFN_QFN:QFN-56-1EP_7x7mm_P0.4mm_EP3.2x3.2mm, F.Cu at (60.1, 59.9)
- added U8: AM26LV32xD, AM26LV32:AM26LV32EIRGYRG4, F.Cu at (58.6, 71.5)
- added U9: LTC2856xDD-1, Package_DFN_QFN:DFN-8-1EP_3x3mm_P0.5mm_EP1.66x2.38mm, F.Cu at (63.5, 70.4)
- added Y1: Crystal_GND24, Crystal:Crystal_SMD_2520-4Pin_2.5x2.0mm, F.Cu at (58.5, 65.8)
- C10, C12, C13, C4, C5, C6, C7, C8, C9, U5: moved to F.Cu
- moved C4 44.2 mm to (47.4, 66.1), turned to 180 degrees
- moved C5 36.2 mm to (51.8, 62.8)
- moved R21 35.6 mm to (52.3, 85.4)
- moved C71 35.6 mm to (59.3, 89.6)
- moved C73 35.6 mm to (59.3, 91.8)
- moved R23 35.6 mm to (55.9, 85.4)
- moved R25 35.6 mm to (55.3, 83.7)
- moved R27 35.6 mm to (57.1, 85.4)
- moved R35 35.6 mm to (52.8, 89.6)
- moved R39 35.6 mm to (52.8, 91.8)
- moved C70 35.6 mm to (55.4, 89.6)
- moved C72 35.6 mm to (55.4, 91.8)
- moved R22 35.6 mm to (52.9, 83.7)
- moved R36 35.6 mm to (54.1, 89.6)
- moved R40 35.6 mm to (54.1, 91.8)
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Routing:
- net +3V3: track 110.5 -> 73.5 mm, vias 17 -> 8
- net +5V: track 12.1 -> 29.7 mm
- net /LIM_AUX: track 15.3 -> 0.00 mm, vias 2 -> 0
- net Lim_R_In: track 14.4 -> 0.00 mm
- net /LIM_H: track 13.5 -> 0.00 mm, vias 2 -> 0
- net /LIM_L: track 12.2 -> 0.00 mm, vias 2 -> 0
- net /LIM_R: track 11.7 -> 0.00 mm, vias 2 -> 0
- net Enc_I_In+: track 14.4 -> 3.50 mm
- net Lim_Aux_In: track 10.4 -> 0.00 mm
- net GND: track 33.6 -> 23.6 mm, vias 200 -> 175
- net Enc_I_In-: track 9.94 -> 1.05 mm
- net Lim_L_In: track 8.63 -> 0.00 mm
- net /PH3_HI: track 9.16 -> 0.97 mm, vias 2 -> 1
- net /HALL_B: track 16.8 -> 9.06 mm
- net /PH3_SENSE: track 43.3 -> 35.6 mm, vias 2 -> 1
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