File: ECE4760 Motor Driver.kicad_sch (KiCad schematic)
At the start: 34 parts, among them J1 IO, J100 Alternative Motor, J2 Motor / Power, J3 USB_B_Micro, J4 UART, J5 Debug, J6 Boot, U1 STM32G473V_B-C-E_Hx, U5 TLV75733PDBV, X1 48MHz

Commit message: Play around with switching to RP2040
Parts:
- removed U1: STM32G473V_B-C-E_Hx, Package_BGA:TFBGA-100_8x8mm_Layout10x10_P0.8mm, symbol MCU_ST_STM32G4:STM32G473V_B-C-E_Hx
- removed X1: 48MHz, Oscillator:Oscillator_SMD_ECS_2520MV-xxx-xx-4Pin_2.5x2.0mm, symbol Oscillator:ECS-2520MV-xxx-xx
- added C74, C75, C76, C77, C78, C79: 100n, Capacitor_SMD:C_0402_1005Metric, symbol Device:C
- added U10: W25Q32JVSS, W25Q:W25Q64JWUUIQTR, symbol Memory_Flash:W25Q32JVSS
- added U7: RP2040, Package_DFN_QFN:QFN-56-1EP_7x7mm_P0.4mm_EP3.2x3.2mm, symbol MCU_RaspberryPi:RP2040
- added U8: AM26LV32xD, AM26LV32:AM26LV32EIRGYRG4, symbol Interface:AM26LV32xD
- added U9: LTC2856xDD-1, Package_DFN_QFN:DFN-8-1EP_3x3mm_P0.5mm_EP1.66x2.38mm, symbol Interface_UART:LTC2856xDD-1
- added Y1: Crystal_GND24, Crystal:Crystal_SMD_2520-4Pin_2.5x2.0mm, symbol Device:Crystal_GND24
Connections:
- net PH1_HI: now also U7.37 (GPIO25)
- net PH1_LO: now also U7.36 (GPIO24)
- net PH1_SENSE: now also U7.41 (GPIO29_ADC3)
- net PH2_HI: now also U7.35 (GPIO23)
- net PH2_LO: now also U7.34 (GPIO22)
- net PH2_SENSE: now also U7.40 (GPIO28_ADC2)
- net PH3_HI: now also U7.32 (GPIO21)
- net PH3_LO: now also U7.31 (GPIO20)
- net PH3_SENSE: now also U7.39 (GPIO27_ADC1)
- net PH4_HI: now also U7.30 (GPIO19)
- net PH4_LO: now also U7.29 (GPIO18)
- net PH4_SENSE: now also U7.38 (GPIO26_ADC0)
- new net: U9.5 (GND), U9.9 (GND)
- new net: U7.1 (IOVDD), U7.10 (IOVDD), U7.22 (IOVDD), U7.33 (IOVDD), U7.42 (IOVDD), U7.49 (IOVDD)
- new net: U7.23 (DVDD), U7.50 (DVDD)
