File: ECE4760 Motor Driver.kicad_sch (KiCad schematic)
At the start: 47 parts, among them J1 IO, J101 Alternative Motor, J2 Motor / Power, J3 UART, U1 STM32G473CETx, U6 AP7361C-33FGE, U7 TPSM365R6, X1 48MHz

Commit message: Update
Parts:
- removed C2: 100n, 100V, 0603, X7R, Capacitor_SMD:C_0603_1608Metric, symbol Device:C
- removed C3: 1u, 100V, 0805, X7R, Capacitor_SMD:C_0805_2012Metric, symbol Device:C
- removed C4, C5: 22u, Capacitor_SMD:C_0805_2012Metric, symbol Device:C
- removed C69, C74, C75, C76, C77, C78, C79, C80, C81, C82, C83, C84: 100n, Capacitor_SMD:C_0402_1005Metric, symbol Device:C
- removed C7, C70, C71, C72, C73: 4u7, Capacitor_SMD:C_0603_1608Metric, symbol Device:C
- removed R1: 40k2, Resistor_SMD:R_0402_1005Metric, symbol Device:R_US
- removed R28, R29: 1k, Resistor_SMD:R_0402_1005Metric, symbol Device:R_US
- removed R3: 10k, Resistor_SMD:R_0402_1005Metric, symbol Device:R_US
- removed TP1: RESET, TestPoint:TestPoint_Pad_D2.0mm, symbol Connector:TestPoint
- removed TP2: BOOT, TestPoint:TestPoint_Pad_D2.0mm, symbol Connector:TestPoint
- removed U7: TPSM365R6, TPSM:RDN0011A-MFG, symbol TPSM:TPSM365R6FRDNR
- added C10, C11: 22u, Capacitor_SMD:C_0805_2012Metric, symbol Device:C
- added C12: 10u, Capacitor_SMD:C_0805_2012Metric, symbol Device:C
- added C13: 100n, Capacitor_SMD:C_0402_1005Metric, symbol Device:C
- added D6: Green, LED_SMD:LED_1206_3216Metric, symbol Device:LED
- added L1: 4u7, Inductor_SMD:L_1008_2520Metric, symbol Device:L
- added R2: 330, Resistor_SMD:R_0402_1005Metric, symbol Device:R_US
- added SW1: RESET, Button_Switch_SMD:SW_SPST_PTS810, symbol Switch:SW_Push
- added U13: AP63205WU, Package_TO_SOT_SMD:TSOT-23-6, symbol Regulator_Switching:AP63205WU
- added U9: MAX13433EETD, Package_DFN_QFN:DFN-14-1EP_3x3mm_P0.4mm_EP1.78x2.35mm, symbol Interface_UART:MAX13433EETD
- C1: footprint Capacitor_SMD:CP_Elec_6.3x7.7 -> Capacitor_THT:CP_Radial_D6.3mm_P2.50mm
- J1: footprint Connector_PinSocket_2.54mm:PinSocket_2x17_P2.54mm_Vertical -> Connector_PinSocket_2.54mm:PinSocket_2x14_P2.54mm_Vertical; symbol Connector_Generic:Conn_02x17_Odd_Even -> Connector_Generic:Conn_02x14_Odd_Even
- J3: footprint Connector_PinHeader_2.54mm:PinHeader_1x05_P2.54mm_Vertical -> Connector_PinHeader_2.54mm:PinHeader_2x04_P2.54mm_Vertical; symbol Connector_Generic:Conn_01x05 -> Connector_Generic:Conn_02x04_Odd_Even
- RV1: value 60V 250A -> 26V 200A; DigiKey F3830CT-ND -> F3823CT-ND; LCSC C2760142 -> C2659457
Connections:
- net Aux_Enc_A_In+ is gone; now on net Hall_C_In: J1.12 (Pin_12)
- net Aux_Enc_A_In- is gone; now on net Hall_I_In: J1.11 (Pin_11)
- net Aux_Enc_B_In+ is gone; now on net Hall_A_In: J1.9 (Pin_9)
- net Aux_Enc_B_In- is gone; now on net Hall_B_In: J1.10 (Pin_10)
- net +3V3: now also U1.1 (VBAT), U1.21 (VDDA), U1.24 (VDD), U1.36 (VDD), U1.48 (VDD); no longer J1.19 (Pin_19)
- net +5V: now also C10.1, C11.1, L1.2, U13.1 (FB); no longer J1.1 (Pin_1), J1.13 (Pin_13), J1.27 (Pin_27), J1.33 (Pin_33), J1.7 (Pin_7)
- net ENC_A+: now also U1.15 (PA7)
- net ENC_A-: now also U1.13 (PA5)
- net ENC_B+: now also U1.16 (PB0)
- net ENC_B-: now also U1.18 (PB2)
- net ENC_I+: now also U1.17 (PB1)
- net ENC_I-: now also U1.12 (PA4)
- net GND: now also J2.6 (Pin_6), J3.5 (Pin_5), J3.6 (Pin_6), J3.8 (Pin_8), U1.19 (VSSA), U1.23 (VSS), U1.35 (VSS), U1.47 (VSS), C10.2, C11.2, C12.2, D6.1 (K), SW1.1, U13.4 (GND), U9.15 (EP), U9.6 (GND), U9.8 (GND); no longer J1.14 (Pin_14), J1.2 (Pin_2), J1.20 (Pin_20), J1.28 (Pin_28), J1.34 (Pin_34), J1.8 (Pin_8), J2.2 (Pin_2), J3.3 (Pin_3)
- net HALL_A: now also U1.8 (PA0)
- net HALL_B: now also U1.9 (PA1)
- net HALL_C: now also U1.10 (PA2)
- net Hall_A_In: no longer J1.29 (Pin_29)
- net Hall_B_In: no longer J1.30 (Pin_30)
- net Hall_C_In: no longer J1.32 (Pin_32)
- net Hall_I_In: no longer J1.31 (Pin_31)
- net LIM_H: now also U1.4 (PC15)
- net LIM_L: now also U1.2 (PC13)
- net LIM_R: now also U1.3 (PC14)
- net OSC_IN: now also U1.5 (PF0)
- net PH1: now also J2.1 (Pin_1); no longer J2.3 (Pin_3)
- net PH1_HI: now also U1.46 (PB9)
- net PH1_LO: now also U1.42 (PB5)
- net PH1_SENSE: now also U1.28 (PB14)
- net PH2: now also J2.2 (Pin_2); no longer J2.4 (Pin_4)
- net PH2_HI: now also U1.32 (PA10)
- net PH2_LO: now also U1.29 (PB15)
- net PH2_SENSE: now also U1.27 (PB13)
- net PH3: now also J2.3 (Pin_3); no longer J2.5 (Pin_5)
- net PH3_HI: now also U1.31 (PA9)
- net PH3_LO: now also U1.34 (PA12)
- net PH3_SENSE: now also U1.26 (PB12)
- net PH4: now also J2.4 (Pin_4); no longer J2.6 (Pin_6)
- net PH4_HI: now also U1.30 (PA8)
- net PH4_LO: now also U1.33 (PA11)
- net PH4_SENSE: now also U1.25 (PB11)
- net SWCLK: now also J3.2 (Pin_2), U1.38 (PA14); no longer J3.5 (Pin_5)
- net SWDIO: now also U1.37 (PA13)
- net UART_RX: now also U1.44 (PB7)
- net UART_TX: now also J3.3 (Pin_3), U1.43 (PB6); no longer J3.2 (Pin_2)
- net Vdrive: now also J2.5 (Pin_5), C12.1, U13.3 (IN); no longer J2.1 (Pin_1)
- net ~{Fault_Enable}: now also U1.39 (PA15); no longer J1.17 (Pin_17)
- net ~{RST}: now also U1.7 (PG10), SW1.2
- net at R30.1: now also U1.14 (PA6); no longer D5.2 (A)
- net at R30.2: now also D5.2 (A)
- net at U1.11 (PA3): now also R2.1
- net at U1.40 (PB3): now also U9.5 (DI)
- net at U1.41 (PB4): now also U9.2 (RO)
- net BOOT: now reaches U1.45 (PB8)
- net BOOT: now also J3.7 (Pin_7)
- net LED_1 renamed CLK+
- net LED_2 renamed CLK-
- net ~{Abort} renamed DATA-
- new net: C13.2, L1.1, U13.5 (SW)
- new net: C13.1, U13.6 (BST)
- new net: D6.2 (A), R2.2
- new net DATA+: J1.17 (Pin_17)
- no-connect marks 31 -> 2
Other:
- removed sheet Encoder Input4
- removed sheet Encoder Input5
- removed sheet Hall Sensor Input4
- removed sheet Limit Switch Input4
- note removed: "Aux Encoder Inputs"
- note removed: "Decoupling capacitors, place close to U1 on all sides"
- note removed: "Unused pins, some connected for routing purposes"
- moved on the sheet: D5, R30

Commit message: Boards ordered!
Parts:
- removed J3: UART, Connector_PinHeader_2.54mm:PinHeader_2x04_P2.54mm_Vertical, symbol Connector_Generic:Conn_02x04_Odd_Even
- removed U9: MAX13433EETD, Package_DFN_QFN:DFN-14-1EP_3x3mm_P0.4mm_EP1.78x2.35mm, symbol Interface_UART:MAX13433EETD
- added C14, C3, C4, C5, C6, C7: 100n, Capacitor_SMD:C_0402_1005Metric, symbol Device:C
- added J1: Comms, Connector_PinHeader_2.54mm:PinHeader_1x05_P2.54mm_Vertical, symbol Connector_Generic:Conn_01x05
- added J3: IO, Connector_PinSocket_2.54mm:PinSocket_2x08_P2.54mm_Vertical, symbol Connector_Generic:Conn_02x08_Odd_Even
- added R1: 330R, Resistor_SMD:R_0402_1005Metric, symbol Device:R_US
- added R2: 4k7, Resistor_SMD:R_0402_1005Metric, symbol Device:R_US
- added SW2: BOOT, Button_Switch_SMD:SW_SPST_PTS810, symbol Switch:SW_Push
- added SW3: POWER, Button_Switch_SMD:SW_SPST_PTS810, symbol Switch:SW_Push
- added SW4: G12JPC, Button_Switch_THT:SW_NKK_G1xJP, symbol Switch:SW_SPST_LED
- added U4: THVD1451D, Package_SO:SOIC-8_3.9x4.9mm_P1.27mm, symbol Interface_UART:THVD1451D
- C1: footprint Capacitor_THT:CP_Radial_D6.3mm_P2.50mm -> Capacitor_THT:CP_Radial_D5.0mm_P2.50mm; DigiKey (none) -> P5190-ND; LCSC C7471882 -> (none)
- C10, C11: LCSC (none) -> C86816
- C12: renamed from C6; DigiKey 490-GRM188Z71C475KE21DCT-ND -> (none); LCSC C389010 -> C437557
- C13: renamed from C8; DigiKey 490-GRM188Z71C475KE21DCT-ND -> (none); LCSC C389010 -> C437557
- C8: renamed from C13; DigiKey (none) -> 490-3261-1-ND; LCSC (none) -> C71629
- C9: renamed from C12; value 10u -> 4u7, 50V; LCSC (none) -> C437557
- D1: renamed from D5; footprint LED_SMD:LED_1206_3216Metric -> LED_SMD:LED_0603_1608Metric; DigiKey 160-2018-1-ND -> (none); LCSC C364563 -> C125101
- D2: renamed from D6; footprint LED_SMD:LED_1206_3216Metric -> LED_SMD:LED_0603_1608Metric; DigiKey 160-2018-1-ND -> (none); LCSC C364563 -> C125101
- J2: renamed from J1; footprint Connector_PinSocket_2.54mm:PinSocket_2x14_P2.54mm_Vertical -> Connector_PinSocket_2.54mm:PinSocket_2x05_P2.54mm_Vertical; symbol Connector_Generic:Conn_02x14_Odd_Even -> Connector_Generic:Conn_02x05_Odd_Even
- L1: DigiKey (none) -> 490-5116-1-ND; LCSC (none) -> C82314
- R3: renamed from R2; value 330 -> 330R; LCSC C138006 -> C105875
- R4: renamed from R30; value 330 -> 330R; LCSC C138006 -> C105875
- RV1: footprint Capacitor_SMD:C_1210_3225Metric -> Capacitor_SMD:C_0603_1608Metric; Comments (none) -> Reduced size for LCSC stock -- reccomend increasing to larg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; DigiKey F3823CT-ND -> (none); LCSC C2659457 -> C2655584
- U1: renamed from U13; LCSC (none) -> C2071056
- U2: renamed from U6; footprint Package_DFN_QFN:DFN-8-1EP_3x3mm_P0.5mm_EP1.65x2.38mm -> Package_DFN_QFN:DFN-8-1EP_3x3mm_P0.65mm_EP1.55x2.4mm
- U3: renamed from U1; LCSC (none) -> C730111
- X1: LCSC C3034286 -> C390534
- renumbered C85 to C2, J101 to J4, J2 to J5
Connections:
- net Lim_Aux_In is gone; now on net +5V: J2.5 (Pin_5)
- net ~{Fault_Enable} is gone; now on net Fault_Enable: U3.39 (PA15)
- net +3V3: now also X1.1 (Tri-State), C14.1, C3.1, C4.1, C5.1, C6.1, C7.1, U4.1 (VCC)
- net +5V: now also J3.13 (Pin_13), J3.15 (Pin_15), J3.3 (Pin_3), J3.5 (Pin_5), R1.2, R2.1
- net BOOT: now also SW2.2
- net CLK+: now also J2.7 (Pin_7), U4.8 (A); no longer J2.15 (Pin_15)
- net CLK-: now also J2.8 (Pin_8), U4.7 (B); no longer J2.16 (Pin_16)
- net DATA+: now also J2.10 (Pin_10), U4.5 (Y); no longer J2.17 (Pin_17)
- net DATA-: now also J2.9 (Pin_9), U4.6 (Z); no longer J2.18 (Pin_18)
- net Enc_A_In+: now also J3.9 (Pin_9); no longer J2.22 (Pin_22)
- net Enc_A_In-: now also J3.10 (Pin_10); no longer J2.21 (Pin_21)
- net Enc_B_In+: now also J3.11 (Pin_11); no longer J2.24 (Pin_24)
- net Enc_B_In-: now also J3.12 (Pin_12); no longer J2.23 (Pin_23)
- net Enc_I_In+: now also J3.7 (Pin_7); no longer J2.26 (Pin_26)
- net Enc_I_In-: now also J3.8 (Pin_8); no longer J2.25 (Pin_25)
- net GND: now also J2.6 (Pin_6), J4.21 (Pin_21), J4.22 (Pin_22), J4.23 (Pin_23), J4.24 (Pin_24), C14.2, C3.2, C4.2, C5.2, C6.2, C7.2, J1.3 (Pin_3), J3.14 (Pin_14), J3.16 (Pin_16), J3.6 (Pin_6), SW2.1, SW3.1, SW4.2 (COM), U4.4 (GND); no longer J4.5 (Pin_5), J4.6 (Pin_6), J4.7 (Pin_7), J4.8 (Pin_8)
- net Hall_A_In: now also J3.2 (Pin_2); no longer J2.9 (Pin_9)
- net Hall_B_In: now also J3.4 (Pin_4); no longer J2.10 (Pin_10)
- net Hall_C_In: now also J3.1 (Pin_1); no longer J2.12 (Pin_12)
- net Lim_H_In: now also J2.2 (Pin_2); no longer J2.6 (Pin_6)
- net PH1: now also J4.1 (Pin_1), J4.2 (Pin_2), J4.3 (Pin_3), J4.4 (Pin_4); no longer J4.10 (Pin_10), J4.11 (Pin_11), J4.12 (Pin_12), J4.9 (Pin_9)
- net PH1_SENSE: now also U3.25 (PB11); no longer U3.28 (PB14)
- net PH2: now also J4.5 (Pin_5), J4.6 (Pin_6), J4.7 (Pin_7), J4.8 (Pin_8); no longer J4.13 (Pin_13), J4.14 (Pin_14), J4.15 (Pin_15), J4.16 (Pin_16)
- net PH2_SENSE: now also U3.26 (PB12); no longer U3.27 (PB13)
- net PH3: now also J4.10 (Pin_10), J4.11 (Pin_11), J4.12 (Pin_12), J4.9 (Pin_9); no longer J4.17 (Pin_17), J4.18 (Pin_18), J4.19 (Pin_19), J4.20 (Pin_20)
- net PH3_SENSE: now also U3.27 (PB13); no longer U3.26 (PB12)
- net PH4: now also J4.13 (Pin_13), J4.14 (Pin_14), J4.15 (Pin_15), J4.16 (Pin_16); no longer J4.21 (Pin_21), J4.22 (Pin_22), J4.23 (Pin_23), J4.24 (Pin_24)
- net PH4_SENSE: now also U3.28 (PB14); no longer U3.25 (PB11)
- net SWCLK: now also J1.2 (Pin_2)
- net SWDIO: now also J1.1 (Pin_1)
- net UART_RX: now also J1.5 (Pin_5)
- net UART_TX: now also J1.4 (Pin_4)
- net Vdrive: now also J4.17 (Pin_17), J4.18 (Pin_18), J4.19 (Pin_19), J4.20 (Pin_20); no longer J4.1 (Pin_1), J4.2 (Pin_2), J4.3 (Pin_3), J4.4 (Pin_4)
- net LED_2: now reaches R4.1, U3.14 (PA6)
- net at U1.2 (EN): now also SW3.2
- net LED_1: now reaches R3.1, U3.11 (PA3)
- net DATA: now reaches U3.41 (PB4)
- net DATA: now also U4.3 (D)
- net CLK: now reaches U3.40 (PB3)
- net CLK: now also U4.2 (R)
- net Fault_Enable: now reaches J2.1 (Pin_1)
- net Fault_Enable: now also R2.2, SW4.3, SW4.6 (K)
- removed net Hall_I_In: J2.11 (Pin_11)
- new net: R1.1, SW4.5 (A)
- no-connect marks 2 -> 1
Other:
- moved on the sheet: C1, C10, C11, C12, C13, C2, C8, C9, D1, D2, J4, J5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
