File: Encoder Input.kicad_sch (KiCad schematic)
At the start: 3 parts

Commit message: Getting ready for fab
Parts:
- R20, R21, R22: DigiKey (none) -> 311-1.00KLRCT-ND
Changed lines of the file:
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@@
     (rev "0")
     (company "Cornell High Energy Synchrotron Source")
+    (comment 1 "Encoder Input Filtering")
     (comment 3 "S. Bywater")
     (comment 4 "S. Bywater")
@@
       (effects (font (size 1.27 1.27)) hide)
     )
+    (property "DigiKey" "311-1.00KLRCT-ND" (at 139.7 101.6 0)
+      (effects (font (size 1.27 1.27)) hide)
+    )
+    (property "LCSC" "" (at 139.7 101.6 0)
+      (effects (font (size 1.27 1.27)) hide)
+    )
     (pin "1")
     (pin "2")
@@
     )
     (property "Comments" "" (at 146.05 95.25 0)
+      (effects (font (size 1.27 1.27)) hide)
+    )
+    (property "DigiKey" "311-1.00KLRCT-ND" (at 146.05 95.25 0)
+      (effects (font (size 1.27 1.27)) hide)
+    )
+    (property "LCSC" "" (at 146.05 95.25 0)
       (effects (font (size 1.27 1.27)) hide)
     )
@@
       (effects (font (size 1.27 1.27)) hide)
     )
+    (property "DigiKey" "311-1.00KLRCT-ND" (at 139.7 88.9 0)
+      (effects (font (size 1.27 1.27)) hide)
+    )
+    (property "LCSC" "" (at 139.7 88.9 0)
+      (effects (font (size 1.27 1.27)) hide)
+    )

Commit message: Ready for design review
Parts:
- R31: renamed from R20; value 1k, 0.1% -> 1k, 1%; LCSC (none) -> C2935237
- R32: renamed from R22; value 1k, 0.1% -> 1k, 1%; LCSC (none) -> C2935237
- R33: renamed from R21; value 1k, 0.1% -> 1k, 1%; LCSC (none) -> C2935237
Changed lines of the file:
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@@
   (symbol (lib_id "Device:R_US") (at 139.7 101.6 90) (unit 1)
     (in_bom yes) (on_board yes) (dnp no)
-    (property "Reference" "R21" (at 139.7 96.52 90)
+    (property "Reference" "R33" (at 139.7 96.52 90)
       (effects (font (size 1.27 1.27)))
     )
-    (property "Value" "1k, 0.1%" (at 139.7 99.06 90)
+    (property "Value" "1k, 1%" (at 139.7 99.06 90)
       (effects (font (size 1.27 1.27)))
     )
@@
       (effects (font (size 1.27 1.27)) hide)
     )
-    (property "LCSC" "" (at 139.7 101.6 0)
+    (property "LCSC" "C2935237" (at 139.7 101.6 0)
       (effects (font (size 1.27 1.27)) hide)
     )
@@
       (project "ECE4760 Motor Driver"
         (path "/6b38a626-de8c-4b2d-bc76-3a02bc823a86/67f78701-eb6f-4714-bcc7-4eb1ac4068c0"
-          (reference "R21") (unit 1)
+          (reference "R33") (unit 1)
         )
         (path "/6b38a626-de8c-4b2d-bc76-3a02bc823a86/dc22c45f-b7c4-46aa-99d2-c66429851554"
-          (reference "R24") (unit 1)
+          (reference "R36") (unit 1)
         )
         (path "/6b38a626-de8c-4b2d-bc76-3a02bc823a86/b169a8bd-422e-4172-a58e-875b2cfce688"
-          (reference "R27") (unit 1)
+          (reference "R39") (unit 1)
         )
         (path "/6b38a626-de8c-4b2d-bc76-3a02bc823a86/f96e87f7-a91c-406f-aa8b-cee643b81ae8"
-          (reference "R30") (unit 1)
+          (reference "R42") (unit 1)
         )
         (path "/6b38a626-de8c-4b2d-bc76-3a02bc823a86/25eb3275-76e1-435c-9a84-78dbb9e1562e"
-          (reference "R33") (unit 1)
+          (reference "R45") (unit 1)
         )
       )
@@
   (symbol (lib_id "Device:R_US") (at 146.05 95.25 180) (unit 1)
     (in_bom yes) (on_board yes) (dnp no) (fields_autoplaced)
-    (property "Reference" "R22" (at 147.955 93.98 0)
+    (property "Reference" "R32" (at 147.955 93.98 0)
       (effects (font (size 1.27 1.27)) (justify right))
     )
-    (property "Value" "1k, 0.1%" (at 147.955 96.52 0)
+    (property "Value" "1k, 1%" (at 147.955 96.52 0)
       (effects (font (size 1.27 1.27)) (justify right))
     )
@@
       (effects (font (size 1.27 1.27)) hide)
     )
-    (property "LCSC" "" (at 146.05 95.25 0)
+    (property "LCSC" "C2935237" (at 146.05 95.25 0)
       (effects (font (size 1.27 1.27)) hide)
     )
@@
       (project "ECE4760 Motor Driver"
         (path "/6b38a626-de8c-4b2d-bc76-3a02bc823a86/67f78701-eb6f-4714-bcc7-4eb1ac4068c0"
-          (reference "R22") (unit 1)
+          (reference "R32") (unit 1)
         )
         (path "/6b38a626-de8c-4b2d-bc76-3a02bc823a86/dc22c45f-b7c4-46aa-99d2-c66429851554"
-          (reference "R25") (unit 1)
+          (reference "R35") (unit 1)
         )
         (path "/6b38a626-de8c-4b2d-bc76-3a02bc823a86/b169a8bd-422e-4172-a58e-875b2cfce688"
-          (reference "R28") (unit 1)
+          (reference "R38") (unit 1)
         )
         (path "/6b38a626-de8c-4b2d-bc76-3a02bc823a86/f96e87f7-a91c-406f-aa8b-cee643b81ae8"
-          (reference "R31") (unit 1)
+          (reference "R41") (unit 1)
         )
         (path "/6b38a626-de8c-4b2d-bc76-3a02bc823a86/25eb3275-76e1-435c-9a84-78dbb9e1562e"
-          (reference "R34") (unit 1)
+          (reference "R44") (unit 1)
         )
       )
@@
   (symbol (lib_id "Device:R_US") (at 139.7 88.9 90) (unit 1)
     (in_bom yes) (on_board yes) (dnp no)
-    (property "Reference" "R20" (at 139.7 83.82 90)
+    (property "Reference" "R31" (at 139.7 83.82 90)
       (effects (font (size 1.27 1.27)))
     )
-    (property "Value" "1k, 0.1%" (at 139.7 86.36 90)
+    (property "Value" "1k, 1%" (at 139.7 86.36 90)
       (effects (font (size 1.27 1.27)))
     )
@@
       (effects (font (size 1.27 1.27)) hide)
     )
-    (property "LCSC" "" (at 139.7 88.9 0)
+    (property "LCSC" "C2935237" (at 139.7 88.9 0)
       (effects (font (size 1.27 1.27)) hide)
     )
@@
       (project "ECE4760 Motor Driver"
         (path "/6b38a626-de8c-4b2d-bc76-3a02bc823a86/67f78701-eb6f-4714-bcc7-4eb1ac4068c0"
-          (reference "R20") (unit 1)
+          (reference "R31") (unit 1)
         )
         (path "/6b38a626-de8c-4b2d-bc76-3a02bc823a86/dc22c45f-b7c4-46aa-99d2-c66429851554"
-          (reference "R23") (unit 1)
+          (reference "R34") (unit 1)
         )
         (path "/6b38a626-de8c-4b2d-bc76-3a02bc823a86/b169a8bd-422e-4172-a58e-875b2cfce688"
-          (reference "R26") (unit 1)
+          (reference "R37") (unit 1)
         )
         (path "/6b38a626-de8c-4b2d-bc76-3a02bc823a86/f96e87f7-a91c-406f-aa8b-cee643b81ae8"
-          (reference "R29") (unit 1)
+          (reference "R40") (unit 1)
         )
         (path "/6b38a626-de8c-4b2d-bc76-3a02bc823a86/25eb3275-76e1-435c-9a84-78dbb9e1562e"
-          (reference "R32") (unit 1)
+          (reference "R43") (unit 1)
         )
       )

Commit message: Boards ordered!
Parts:
- R19: renamed from R31; LCSC C2935237 -> C242161
- R20: renamed from R32; LCSC C2935237 -> C242161
- R21: renamed from R33; LCSC C2935237 -> C242161
Changed lines of the file:
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@@
   (symbol (lib_id "Device:R_US") (at 139.7 101.6 90) (unit 1)
     (in_bom yes) (on_board yes) (dnp no)
-    (property "Reference" "R33" (at 139.7 96.52 90)
+    (property "Reference" "R21" (at 139.7 96.52 90)
       (effects (font (size 1.27 1.27)))
     )
@@
       (effects (font (size 1.27 1.27)) hide)
     )
-    (property "LCSC" "C2935237" (at 139.7 101.6 0)
+    (property "LCSC" "C242161" (at 139.7 101.6 0)
       (effects (font (size 1.27 1.27)) hide)
     )
@@
       (project "ECE4760 Motor Driver"
         (path "/6b38a626-de8c-4b2d-bc76-3a02bc823a86/67f78701-eb6f-4714-bcc7-4eb1ac4068c0"
-          (reference "R33") (unit 1)
+          (reference "R21") (unit 1)
         )
         (path "/6b38a626-de8c-4b2d-bc76-3a02bc823a86/dc22c45f-b7c4-46aa-99d2-c66429851554"
-          (reference "R36") (unit 1)
+          (reference "R24") (unit 1)
         )
         (path "/6b38a626-de8c-4b2d-bc76-3a02bc823a86/b169a8bd-422e-4172-a58e-875b2cfce688"
-          (reference "R39") (unit 1)
+          (reference "R27") (unit 1)
         )
       )
@@
   (symbol (lib_id "Device:R_US") (at 146.05 95.25 180) (unit 1)
     (in_bom yes) (on_board yes) (dnp no) (fields_autoplaced)
-    (property "Reference" "R32" (at 147.955 93.98 0)
+    (property "Reference" "R20" (at 147.955 93.98 0)
       (effects (font (size 1.27 1.27)) (justify right))
     )
@@
       (effects (font (size 1.27 1.27)) hide)
     )
-    (property "LCSC" "C2935237" (at 146.05 95.25 0)
+    (property "LCSC" "C242161" (at 146.05 95.25 0)
       (effects (font (size 1.27 1.27)) hide)
     )
@@
       (project "ECE4760 Motor Driver"
         (path "/6b38a626-de8c-4b2d-bc76-3a02bc823a86/67f78701-eb6f-4714-bcc7-4eb1ac4068c0"
-          (reference "R32") (unit 1)
+          (reference "R20") (unit 1)
         )
         (path "/6b38a626-de8c-4b2d-bc76-3a02bc823a86/dc22c45f-b7c4-46aa-99d2-c66429851554"
-          (reference "R35") (unit 1)
+          (reference "R23") (unit 1)
         )
         (path "/6b38a626-de8c-4b2d-bc76-3a02bc823a86/b169a8bd-422e-4172-a58e-875b2cfce688"
-          (reference "R38") (unit 1)
+          (reference "R26") (unit 1)
         )
       )
@@
   (symbol (lib_id "Device:R_US") (at 139.7 88.9 90) (unit 1)
     (in_bom yes) (on_board yes) (dnp no)
-    (property "Reference" "R31" (at 139.7 83.82 90)
+    (property "Reference" "R19" (at 139.7 83.82 90)
       (effects (font (size 1.27 1.27)))
     )
@@
       (effects (font (size 1.27 1.27)) hide)
     )
-    (property "LCSC" "C2935237" (at 139.7 88.9 0)
+    (property "LCSC" "C242161" (at 139.7 88.9 0)
       (effects (font (size 1.27 1.27)) hide)
     )
@@
       (project "ECE4760 Motor Driver"
         (path "/6b38a626-de8c-4b2d-bc76-3a02bc823a86/67f78701-eb6f-4714-bcc7-4eb1ac4068c0"
-          (reference "R31") (unit 1)
+          (reference "R19") (unit 1)
         )
         (path "/6b38a626-de8c-4b2d-bc76-3a02bc823a86/dc22c45f-b7c4-46aa-99d2-c66429851554"
-          (reference "R34") (unit 1)
+          (reference "R22") (unit 1)
         )
         (path "/6b38a626-de8c-4b2d-bc76-3a02bc823a86/b169a8bd-422e-4172-a58e-875b2cfce688"
-          (reference "R37") (unit 1)
+          (reference "R25") (unit 1)
         )
       )
